File: pcb/usb_relay_hub.kicad_pcb (KiCad board)
At the start: 2 copper layers, 67.9 x 82.5 mm, 80 parts, among them J1 USB2.0_C_v3-R, J2 USB2.0_C_v3-R, J3 USB2.0_C_v3-R, J4 USB2.0_C_v3-R, J5 Power, J6 Com, J7 Com, J8 Com, J9 Com, K1 FINDER-30.22, K2 FINDER-30.22, K3 FINDER-30.22, K4 FINDER-30.22, M1 M2_v2, M2 M2_v2, M3 M2_v2, M4 M2_v2, SW1 SW_Push, SW2 SW_Push, SW3 SW_Push, SW4 SW_Push, U1 CH213K, U10 CH217K, U11 CH334R, U2 CH213K, U3 CH213K, U4 CH213K, U5 AMS1117-3.3, U6 CH32V003F4P6, U7 CH217K, U8 CH217K, U9 CH217K, Y1 12M

Commit message: switch/1.0.0
Parts:
- removed U5: AMS1117-3.3, Package_TO_SOT_SMD:SOT-89-3_Handsoldering
- R21, R22: value 10k -> 1k
Connections:
- C1 pad 1: +3V3 -> +5V
- C2 pad 1: +3V3 -> +5V
- CH2 pad 3: +3V3 -> +5V
- R12 pad 1: +3V3 -> +5V
- R21 pad 1: +3V3 -> +5V
- R22 pad 1: +3V3 -> +5V
- U6 pad 9: +3V3 -> +5V
Routing:
- net +3V3: track 94.1 -> 0.00 mm, vias 2 -> 0
- net +5V: track 124.2 -> 213.3 mm, vias 8 -> 10
- net Net-(R12-Pad2): track 102.9 -> 97.9 mm
- net /BTN4: track 68.8 -> 67.3 mm
- net /SELECT_U2: track 41.2 -> 40.0 mm
- net Net-(U11-XI): track 9.88 -> 8.75 mm
- net /DPU4+: track 20.9 -> 20.1 mm
- net /SWDIO: track 6.90 -> 6.12 mm
- net /DMU2-: track 20.8 -> 20.1 mm
- net /DPU3+: track 21.1 -> 20.5 mm
- net /SELECT_U1: track 27.5 -> 26.9 mm
- net /BTN2: track 33.1 -> 32.5 mm
- net /BTN1: track 16.6 -> 16.0 mm
- net /BTN3: track 50.7 -> 50.1 mm
- net /SDA: track 54.4 -> 53.8 mm
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Other:
- board text added: "Relay USB Switch Hub by 74th v1.0.1"
- board text removed: "Relay USB Switch Hub by 74th v1.0.0"
