File: pcb/usb_relay_hub.kicad_sch (KiCad schematic)
At the start: 74 parts, among them J1 USB2.0_C_v3-R, J2 USB2.0_C_v3-R, J3 USB2.0_C_v3-R, J4 USB2.0_C_v3-R, J5 Power, J6 Com, J7 Com, J8 Com, J9 Com, K1 FINDER-30.22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

Commit message: switch/1.0.0
Parts:
- removed R27: 0, $74th:Register_0603_1608, symbol Device:R
- removed U5: AMS1117-3.3, Package_TO_SOT_SMD:SOT-89-3_Handsoldering, symbol Regulator_Linear:AMS1117-3.3
Connections:
- net +3V3 is gone; now on net +5V: C1.1, C2.1, CH2.3 (VCC), R12.1, R21.1, R22.1, U6.9 (VDD)
- net +5V: now also C8.1, U11.12 (V5)
