File: main-pcb/usb_relay_hub.kicad_sch (KiCad schematic)
At the start: 72 parts, among them J1 USB2.0_C_v3-R, J2 USB2.0_C_v3-R, J3 USB2.0_C_v3-R, J4 USB2.0_C_v3-R, J5 Power, J6 Com, J7 Com, J8 Com, J9 Com, K1 FINDER-30.22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

Commit message: update readme
Parts:
- K1, K2, K3, K4: value FINDER-30.22 -> 941H-2C-5D
Other:
- title: (none) -> Relay USB Switch Hub by 74th
Changed lines of the file:
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@@
 (kicad_sch (version 20230121) (generator eeschema)
   (paper "A3")
+  (title_block
+    (title "Relay USB Switch Hub by 74th")
+  )
   (junction (at 53.34 245.11) (diameter 0) (color 0 0 0 0)
   )
@@
       (effects (font (size 1.27 1.27)))
     )
-    (property "Value" "FINDER-30.22" (at 256.54 93.98 90)
+    (property "Value" "941H-2C-5D" (at 256.54 93.98 90)
       (effects (font (size 1.27 1.27)))
     )
@@
       (effects (font (size 1.27 1.27)))
     )
-    (property "Value" "FINDER-30.22" (at 256.54 33.02 90)
+    (property "Value" "941H-2C-5D" (at 256.54 33.02 90)
       (effects (font (size 1.27 1.27)))
     )
@@
       (effects (font (size 1.27 1.27)))
     )
-    (property "Value" "FINDER-30.22" (at 256.54 210.82 90)
+    (property "Value" "941H-2C-5D" (at 256.54 210.82 90)
       (effects (font (size 1.27 1.27)))
     )
@@
       (effects (font (size 1.27 1.27)))
     )
-    (property "Value" "FINDER-30.22" (at 256.54 151.13 90)
+    (property "Value" "941H-2C-5D" (at 256.54 151.13 90)
       (effects (font (size 1.27 1.27)))
     )
