File: remote_switch-pcb/switch-pcb.kicad_sch (KiCad schematic)
At the start: 15 parts, among them SW1 SW_Push, SW2 SW_Push, SW3 SW_Push, SW4 SW_Push, U1 CH32V003F4P6

Commit message: update readme
Other:
- title: (none) -> Button Unit Grove I2C
Changed lines of the file:
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@@
 (kicad_sch (version 20230121) (generator eeschema)
   (paper "A4")
+  (title_block
+    (title "Button Unit Grove I2C")
+  )
   (junction (at 217.17 48.26) (diameter 0) (color 0 0 0 0)
   )
